Commit message: Adapt to new configuration

File: ur_description/urdf/ur_macro.xacro (robot description, xacro)
@@ -129,5 +129,20 @@
     <!-- Placeholder for ros2_control transmission which don't yet exist -->
     <!-- links -  main serial chain -->
-    <link name="${tf_prefix}base_link"/>
+    <link name="${tf_prefix}base_link">
+      <visual>
+        <origin xyz="0 0 0" rpy="0 0 0"/>
+        <geometry>
+          <mesh filename="package://ur_description/meshes/ur3/bench_simplified.stl"/>
+        </geometry>
+        <material name="blue">
+          <color rgba="${106/255} ${165/255} ${219/255} 1.0"/>        </material>
+      </visual>
+      <collision>
+        <origin xyz="0 0 0" rpy="0 0 0"/>
+        <geometry>
+          <mesh filename="package://ur_description/meshes/ur3/bench_simplified.stl"/>
+        </geometry>
+      </collision>
+    </link>
     <link name="${tf_prefix}base_link_inertia">
       <visual>
@@ -267,5 +282,6 @@
            link/frame) to introduce the necessary rotation over Z (of pi rad).
       -->
-      <origin xyz="0 0 0" rpy="0 0 ${pi}" />
+      <!-- <origin xyz="0 0 0" rpy="0 0 ${pi}" /> -->
+      <origin xyz="0.135 0.0674839772410001 1.241072164125" rpy="${pi} 0 ${2*pi}" />
     </joint>
     <joint name="${tf_prefix}shoulder_pan_joint" type="revolute">

Commit message: Plan with PILZ planner

File: ur_description/urdf/ur_macro.xacro (robot description, xacro)
@@ -283,5 +283,6 @@
       -->
       <!-- <origin xyz="0 0 0" rpy="0 0 ${pi}" /> -->
-      <origin xyz="0.135 0.0674839772410001 1.241072164125" rpy="${pi} 0 ${2*pi}" />
+      <!-- <origin xyz="0.135 0.0674839772410001 1.241072164125" rpy="${pi} 0 ${2*pi}" /> -->
+      <origin xyz="-0.135 0.0674839772410001 1.241072164125" rpy="${pi} 0 ${2*pi}" />
     </joint>
     <joint name="${tf_prefix}shoulder_pan_joint" type="revolute">

Commit message: Correct vention table height to avoid collision

File: ur_description/urdf/ur_macro.xacro (robot description, xacro)
@@ -133,5 +133,5 @@
         <origin xyz="0 0 0" rpy="0 0 0"/>
         <geometry>
-          <mesh filename="package://ur_description/meshes/ur3/bench_simplified.stl"/>
+          <mesh filename="package://ur_description/meshes/ur3/bench_simplified_corrected.stl"/>
         </geometry>
         <material name="blue">
@@ -141,5 +141,5 @@
         <origin xyz="0 0 0" rpy="0 0 0"/>
         <geometry>
-          <mesh filename="package://ur_description/meshes/ur3/bench_simplified.stl"/>
+          <mesh filename="package://ur_description/meshes/ur3/bench_simplified_corrected.stl"/>
         </geometry>
       </collision>
@@ -252,5 +252,5 @@
 	  <xacro:get_visual_params name="wrist_3" type="visual_offset"/>
       <visual>
-        <origin xyz="0 0 ${visual_params}" rpy="${pi/2} 0 0"/>
+        <origin xyz="0 0 ${visual_params}" rpy="${pi} 0 ${pi}"/>
         <geometry>
           <xacro:get_mesh name="wrist_3" type="visual"/>
@@ -284,5 +284,5 @@
       <!-- <origin xyz="0 0 0" rpy="0 0 ${pi}" /> -->
       <!-- <origin xyz="0.135 0.0674839772410001 1.241072164125" rpy="${pi} 0 ${2*pi}" /> -->
-      <origin xyz="-0.135 0.0674839772410001 1.241072164125" rpy="${pi} 0 ${2*pi}" />
+      <origin xyz="-0.135 0.0674839772410001 1.336622164125" rpy="${pi} 0 ${2*pi}" />
     </joint>
     <joint name="${tf_prefix}shoulder_pan_joint" type="revolute">
