Commit message: Correct ur_description version from rolling to humble
The incorrect version of ur_description is being used. It's for ros2 rolling and hence cannot use the flag use_fake_hardware to switch on mock hardware.

File: ur_description/urdf/ur.ros2_control.xacro (robot description, xacro)
@@ -3,5 +3,5 @@
   <xacro:macro name="ur_ros2_control" params="
     name
-    use_fake_hardware:=false fake_sensor_commands:=false
+    use_mock_hardware:=false mock_sensor_commands:=false
     sim_gazebo:=false
     sim_ignition:=false
@@ -19,5 +19,5 @@
     script_command_port:=50004
     trajectory_port:=50003
-    non_blocking_read:=true
+    non_blocking_read:=false
     keep_alive_count:=2
     ">
@@ -30,10 +30,10 @@
           <plugin>ign_ros2_control/IgnitionSystem</plugin>
         </xacro:if>
-        <xacro:if value="${use_fake_hardware}">
+        <xacro:if value="${use_mock_hardware}">
           <plugin>mock_components/GenericSystem</plugin>
-          <param name="fake_sensor_commands">${fake_sensor_commands}</param>
+          <param name="mock_sensor_commands">${mock_sensor_commands}</param>
           <param name="state_following_offset">0.0</param>
         </xacro:if>
-        <xacro:unless value="${use_fake_hardware or sim_gazebo or sim_ignition}">
+        <xacro:unless value="${use_mock_hardware or sim_gazebo or sim_ignition}">
           <plugin>ur_robot_driver/URPositionHardwareInterface</plugin>
           <param name="robot_ip">${robot_ip}</param>
@@ -74,9 +74,13 @@
         </command_interface>
         <state_interface name="position">
-          <!-- initial position for the FakeSystem and simulation -->
+          <!-- initial position for the mock system and simulation -->
           <param name="initial_value">${initial_positions['shoulder_pan_joint']}</param>
         </state_interface>
-        <state_interface name="velocity"/>
-        <state_interface name="effort"/>
+        <state_interface name="velocity">
+          <param name="initial_value">0.0</param>
+        </state_interface>
+        <state_interface name="effort">
+          <param name="initial_value">0.0</param>
+        </state_interface>
       </joint>
       <joint name="${tf_prefix}shoulder_lift_joint">
@@ -90,9 +94,13 @@
         </command_interface>
         <state_interface name="position">
-          <!-- initial position for the FakeSystem and simulation -->
+          <!-- initial position for the mock system and simulation -->
           <param name="initial_value">${initial_positions['shoulder_lift_joint']}</param>
         </state_interface>
-        <state_interface name="velocity"/>
-        <state_interface name="effort"/>
+        <state_interface name="velocity">
+          <param name="initial_value">0.0</param>
+        </state_interface>
+        <state_interface name="effort">
+          <param name="initial_value">0.0</param>
+        </state_interface>
       </joint>
       <joint name="${tf_prefix}elbow_joint">
@@ -106,9 +114,13 @@
         </command_interface>
         <state_interface name="position">
-          <!-- initial position for the FakeSystem and simulation -->
+          <!-- initial position for the mock system and simulation -->
           <param name="initial_value">${initial_positions['elbow_joint']}</param>
         </state_interface>
-        <state_interface name="velocity"/>
-        <state_interface name="effort"/>
+        <state_interface name="velocity">
+          <param name="initial_value">0.0</param>
+        </state_interface>
+        <state_interface name="effort">
+          <param name="initial_value">0.0</param>
+        </state_interface>
       </joint>
       <joint name="${tf_prefix}wrist_1_joint">
@@ -122,9 +134,13 @@
         </command_interface>
         <state_interface name="position">
-          <!-- initial position for the FakeSystem and simulation -->
+          <!-- initial position for the mock system and simulation -->
           <param name="initial_value">${initial_positions['wrist_1_joint']}</param>
         </state_interface>
-        <state_interface name="velocity"/>
-        <state_interface name="effort"/>
+        <state_interface name="velocity">
+          <param name="initial_value">0.0</param>
+        </state_interface>
+        <state_interface name="effort">
+          <param name="initial_value">0.0</param>
+        </state_interface>
       </joint>
       <joint name="${tf_prefix}wrist_2_joint">
@@ -138,9 +154,13 @@
         </command_interface>
         <state_interface name="position">
-          <!-- initial position for the FakeSystem and simulation -->
+          <!-- initial position for the mock system and simulation -->
           <param name="initial_value">${initial_positions['wrist_2_joint']}</param>
         </state_interface>
-        <state_interface name="velocity"/>
-        <state_interface name="effort"/>
+        <state_interface name="velocity">
+          <param name="initial_value">0.0</param>
+        </state_interface>
+        <state_interface name="effort">
+          <param name="initial_value">0.0</param>
+        </state_interface>
       </joint>
       <joint name="${tf_prefix}wrist_3_joint">
@@ -154,9 +174,13 @@
         </command_interface>
         <state_interface name="position">
-          <!-- initial position for the FakeSystem and simulation -->
+          <!-- initial position for the mock system and simulation -->
           <param name="initial_value">${initial_positions['wrist_3_joint']}</param>
         </state_interface>
-        <state_interface name="velocity"/>
-        <state_interface name="effort"/>
+        <state_interface name="velocity">
+          <param name="initial_value">0.0</param>
+        </state_interface>
+        <state_interface name="effort">
+          <param name="initial_value">0.0</param>
+        </state_interface>
       </joint>
       <xacro:unless value="${sim_gazebo or sim_ignition}">
@@ -169,5 +193,5 @@
           <state_interface name="torque.z"/>
         </sensor>
-        <!-- NOTE The following are joints used only for testing with fake hardware and will change in the future -->
+        <!-- NOTE The following are joints used only for testing with mock hardware and will change in the future -->
         <gpio name="${tf_prefix}speed_scaling">
           <state_interface name="speed_scaling_factor"/>

File: ur_description/urdf/ur.urdf.xacro (robot description, xacro)
@@ -40,10 +40,10 @@
    <xacro:arg name="tool_tcp_port" default="54321" />
      <!-- Simulation parameters -->
-   <xacro:arg name="use_fake_hardware" default="false" />
-   <xacro:arg name="fake_sensor_commands" default="false" />
+   <xacro:arg name="use_mock_hardware" default="false" />
+   <xacro:arg name="mock_sensor_commands" default="false" />
    <xacro:arg name="sim_gazebo" default="false" />
    <xacro:arg name="sim_ignition" default="false" />
    <xacro:arg name="simulation_controllers" default="" />
-   <!-- initial position for simulations (Fake Hardware, Gazebo, Ignition) -->
+   <!-- initial position for simulations (Mock Hardware, Gazebo, Ignition) -->
    <xacro:arg name="initial_positions_file" default="$(find ur_description)/config/initial_positions.yaml"/>
    <!-- convert to property to use substitution in function -->
@@ -64,6 +64,6 @@
      safety_pos_margin="$(arg safety_pos_margin)"
      safety_k_position="$(arg safety_k_position)"
-     use_fake_hardware="$(arg use_fake_hardware)"
-     fake_sensor_commands="$(arg fake_sensor_commands)"
+     use_mock_hardware="$(arg use_mock_hardware)"
+     mock_sensor_commands="$(arg mock_sensor_commands)"
      sim_gazebo="$(arg sim_gazebo)"
      sim_ignition="$(arg sim_ignition)"

File: ur_description/urdf/ur_macro.xacro (robot description, xacro)
@@ -53,11 +53,10 @@
     physical_parameters_file
     visual_parameters_file
-    generate_ros2_control_tag:=true
     transmission_hw_interface:=hardware_interface/PositionJointInterface
     safety_limits:=false
     safety_pos_margin:=0.15
     safety_k_position:=20
-    use_fake_hardware:=false
-    fake_sensor_commands:=false
+    use_mock_hardware:=false
+    mock_sensor_commands:=false
     sim_gazebo:=false
     sim_ignition:=false
@@ -82,5 +81,5 @@
     script_command_port:=50004
     trajectory_port:=50003
-    non_blocking_read:=true
+    non_blocking_read:=false
     keep_alive_count:=2"
     >
@@ -92,45 +91,58 @@
       visual_parameters_file="${visual_parameters_file}"
       force_abs_paths="${sim_gazebo or sim_ignition}"/>
-    <xacro:if value="${generate_ros2_control_tag}">
-      <!-- ros2 control include -->
-      <xacro:include filename="$(find ur_description)/urdf/ur.ros2_control.xacro" />
-      <!-- ros2 control instance -->
-      <xacro:ur_ros2_control
-        name="${name}"
-        use_fake_hardware="${use_fake_hardware}"
-        initial_positions="${initial_positions}"
-        fake_sensor_commands="${fake_sensor_commands}"
-        headless_mode="${headless_mode}"
-        sim_gazebo="${sim_gazebo}"
-        sim_ignition="${sim_ignition}"
-        script_filename="${script_filename}"
-        output_recipe_filename="${output_recipe_filename}"
-        input_recipe_filename="${input_recipe_filename}"
-        tf_prefix="${tf_prefix}"
-        hash_kinematics="${kinematics_hash}"
-        robot_ip="${robot_ip}"
-        use_tool_communication="${use_tool_communication}"
-        tool_voltage="${tool_voltage}"
-        tool_parity="${tool_parity}"
-        tool_baud_rate="${tool_baud_rate}"
-        tool_stop_bits="${tool_stop_bits}"
-        tool_rx_idle_chars="${tool_rx_idle_chars}"
-        tool_tx_idle_chars="${tool_tx_idle_chars}"
-        tool_device_name="${tool_device_name}"
-        tool_tcp_port="${tool_tcp_port}"
-        reverse_port="${reverse_port}"
-        script_sender_port="${script_sender_port}"
-        reverse_ip="${reverse_ip}"
-        script_command_port="${script_command_port}"
-        trajectory_port="${trajectory_port}"
-        non_blocking_read="${non_blocking_read}"
-        keep_alive_count="${keep_alive_count}"
-        />
-    </xacro:if>
+    <!-- ros2 control include -->
+    <xacro:include filename="$(find ur_description)/urdf/ur.ros2_control.xacro" />
+    <!-- ros2 control instance -->
+    <xacro:ur_ros2_control
+      name="${name}"
+      use_mock_hardware="${use_mock_hardware}"
+      initial_positions="${initial_positions}"
+      mock_sensor_commands="${mock_sensor_commands}"
+      headless_mode="${headless_mode}"
+      sim_gazebo="${sim_gazebo}"
+      sim_ignition="${sim_ignition}"
+      script_filename="${script_filename}"
+      output_recipe_filename="${output_recipe_filename}"
+      input_recipe_filename="${input_recipe_filename}"
+      tf_prefix="${tf_prefix}"
+      hash_kinematics="${kinematics_hash}"
+      robot_ip="${robot_ip}"
+      use_tool_communication="${use_tool_communication}"
+      tool_voltage="${tool_voltage}"
+      tool_parity="${tool_parity}"
+      tool_baud_rate="${tool_baud_rate}"
+      tool_stop_bits="${tool_stop_bits}"
+      tool_rx_idle_chars="${tool_rx_idle_chars}"
+      tool_tx_idle_chars="${tool_tx_idle_chars}"
+      tool_device_name="${tool_device_name}"
+      tool_tcp_port="${tool_tcp_port}"
+      reverse_port="${reverse_port}"
+      script_sender_port="${script_sender_port}"
+      reverse_ip="${reverse_ip}"
+      script_command_port="${script_command_port}"
+      trajectory_port="${trajectory_port}"
+      non_blocking_read="${non_blocking_read}"
+      keep_alive_count="${keep_alive_count}"
+      />
     <!-- Add URDF transmission elements (for ros_control) -->
     <!--<xacro:ur_arm_transmission prefix="${prefix}" hw_interface="${transmission_hw_interface}" />-->
     <!-- Placeholder for ros2_control transmission which don't yet exist -->
     <!-- links -  main serial chain -->
-    <link name="${tf_prefix}base_link"/>
+    <link name="${tf_prefix}base_link">
+      <visual>
+        <origin xyz="0 0 0" rpy="0 0 0"/>
+        <geometry>
+          <mesh filename="package://ur_description/meshes/ur3/bench_simplified_corrected.stl"/>
+        </geometry>
+        <material name="blue">
+          <color rgba="${106/255} ${165/255} ${219/255} 1.0"/>        </material>
+      </visual>
+      <collision>
+        <origin xyz="0 0 0" rpy="0 0 0"/>
+        <geometry>
+          <mesh filename="package://ur_description/meshes/ur3/bench_simplified_corrected.stl"/>
+        </geometry>
+      </collision>
+    </link>
     <link name="${tf_prefix}base_link_inertia">
       <visual>
@@ -240,5 +252,5 @@
 	  <xacro:get_visual_params name="wrist_3" type="visual_offset"/>
       <visual>
-        <origin xyz="0 0 ${visual_params}" rpy="${pi/2} 0 0"/>
+        <origin xyz="0 0 ${visual_params}" rpy="${pi} 0 ${pi}"/>
         <geometry>
           <xacro:get_mesh name="wrist_3" type="visual"/>
@@ -270,5 +282,7 @@
            link/frame) to introduce the necessary rotation over Z (of pi rad).
       -->
-      <origin xyz="0 0 0" rpy="0 0 ${pi}" />
+      <!-- <origin xyz="0 0 0" rpy="0 0 ${pi}" /> -->
+      <!-- <origin xyz="0.135 0.0674839772410001 1.241072164125" rpy="${pi} 0 ${2*pi}" /> -->
+      <origin xyz="-0.135 0.0674839772410001 1.336622164125" rpy="${pi} 0 ${2*pi}" />
     </joint>
     <joint name="${tf_prefix}shoulder_pan_joint" type="revolute">
