Commit message: Update description package

File: ur_description/urdf/ur.urdf.xacro (robot description, xacro)
@@ -7,5 +7,5 @@
    <!-- possible 'ur_type' values: ur3, ur3e, ur5, ur5e, ur10, ur10e, ur16e, ur20 -->
    <!-- the default value should raise an error in case this was called without defining the type -->
-   <xacro:arg name="ur_type" default="ur5x"/>
+   <xacro:arg name="ur_type" default="ur3"/>
    <!-- parameters -->
    <xacro:arg name="tf_prefix" default="" />
@@ -40,20 +40,40 @@
    <xacro:arg name="tool_tcp_port" default="54321" />
      <!-- Simulation parameters -->
-   <xacro:arg name="use_mock_hardware" default="false" />
-   <xacro:arg name="mock_sensor_commands" default="false" />
+   <xacro:arg name="use_fake_hardware" default="false" />
+   <xacro:arg name="fake_sensor_commands" default="false" />
    <xacro:arg name="sim_gazebo" default="false" />
    <xacro:arg name="sim_ignition" default="false" />
    <xacro:arg name="simulation_controllers" default="" />
-   <!-- initial position for simulations (Mock Hardware, Gazebo, Ignition) -->
+   <!-- initial position for simulations (Fake Hardware, Gazebo, Ignition) -->
    <xacro:arg name="initial_positions_file" default="$(find ur_description)/config/initial_positions.yaml"/>
    <!-- convert to property to use substitution in function -->
    <xacro:property name="initial_positions_file" default="$(arg initial_positions_file)"/>
    <!-- create link fixed to the "world" -->
-   <link name="world" />
+   <!-- <link name="world" /> -->
+   <link name="vention_base">
+    <visual>
+     <origin
+      xyz="0 0 0" rpy="0 0 0" />
+     <geometry>
+      <mesh filename="package://ur_description/meshes/ur3/bench_simplified_corrected.stl" />
+     </geometry>
+     <material name="">
+       <color rgba="${106/255} ${165/255} ${219/255} 1.0" />
+     </material>
+    </visual>
+    <collision>
+     <origin
+      xyz="0 0 0" rpy="0 0 0" />
+     <geometry>
+      <mesh filename="package://ur_description/meshes/ur3/bench_simplified_corrected.stl" />
+     </geometry>
+    </collision>
+   </link>
+   <link name="base_link_dummy"/>
    <!-- arm -->
    <xacro:ur_robot
      name="$(arg name)"
      tf_prefix="$(arg tf_prefix)"
-     parent="world"
+     parent="base_link_dummy"
      joint_limits_parameters_file="$(arg joint_limit_params)"
      kinematics_parameters_file="$(arg kinematics_params)"
@@ -64,6 +84,6 @@
      safety_pos_margin="$(arg safety_pos_margin)"
      safety_k_position="$(arg safety_k_position)"
-     use_mock_hardware="$(arg use_mock_hardware)"
-     mock_sensor_commands="$(arg mock_sensor_commands)"
+     use_fake_hardware="$(arg use_fake_hardware)"
+     fake_sensor_commands="$(arg fake_sensor_commands)"
      sim_gazebo="$(arg sim_gazebo)"
      sim_ignition="$(arg sim_ignition)"
@@ -89,6 +109,12 @@
      trajectory_port="$(arg trajectory_port)"
      >
-     <origin xyz="0 0 0" rpy="0 0 0" />          <!-- position robot in the world -->
+     <origin xyz="0 0 0" rpy="0 0 0" />
+     <!-- <origin xyz="-0.135 0.0674839772410001 1.336622164125" rpy="${pi} 0 ${2*pi}" /> -->
    </xacro:ur_robot>
+   <joint name="vention_base-dummy_link" type="fixed">
+    <parent link="vention_base"/>
+    <child link="base_link_dummy"/>
+    <origin xyz="-0.135 0.0674839772410001 1.336622164125" rpy="${pi} 0 ${pi}" />
+   </joint>
    <xacro:if value="$(arg sim_gazebo)">
     <!-- Gazebo plugins -->
