Commit message: Rename arm_0 and arm_1 to left and right respectively

File: dual_ur_desription/urdf/ur.urdf.xacro (robot description, xacro)
@@ -70,11 +70,11 @@
     </collision>
    </link>
-   <link name = "arm_0_base_link_z"/>
-   <link name = "arm_1_base_link_z"/>
+   <link name = "left_base_link_z"/>
+   <link name = "right_base_link_z"/>
    <!-- arm -->
    <xacro:ur_robot
-     name="arm_0"
-     tf_prefix="arm_0_"
-     parent="arm_0_base_link_z"
+     name="left"
+     tf_prefix="left_"
+     parent="left_base_link_z"
      joint_limits_parameters_file="$(arg joint_limit_params)"
      kinematics_parameters_file="$(arg kinematics_params)"
@@ -113,7 +113,7 @@
    </xacro:ur_robot>
   <xacro:ur_robot
-   name="arm_1"
-   tf_prefix="arm_1_"
-   parent="arm_1_base_link_z"
+   name="right"
+   tf_prefix="right_"
+   parent="right_base_link_z"
    joint_limits_parameters_file="$(arg joint_limit_params)"
    kinematics_parameters_file="$(arg kinematics_params)"
@@ -156,22 +156,22 @@
     <origin xyz="-0.135 0.0674839772410001 1.336622164125" rpy="${pi} 0 ${pi}" />
    </joint> -->
-   <joint name="vention_base-arm_0_base_link_z" type="fixed">
+   <joint name="vention_base-left_base_link_z" type="fixed">
     <parent link="vention_base" />
-    <child link="arm_0_base_link_z" />
+    <child link="left_base_link_z" />
     <origin xyz="-0.135 0.0674839772410001 1.336622164125" rpy="${pi} 0 ${pi}" />
   </joint>
-  <joint name="arm_0_base_link_z-joint_0" type="fixed">
-    <parent link="arm_0_base_link_z" />
-    <child link="arm_0_base_link" />
+  <joint name="left_base_link_z-joint_0" type="fixed">
+    <parent link="left_base_link_z" />
+    <child link="left_base_link" />
     <origin xyz="0 0 0" rpy="0 0 0" />
   </joint>
-  <joint name="vention_base-arm_1_base_link_z" type="fixed">
+  <joint name="vention_base-right_base_link_z" type="fixed">
     <parent link="vention_base" />
-    <child link="arm_1_base_link_z" />
+    <child link="right_base_link_z" />
     <origin xyz="0.135 0.0674839772410001 1.336622164125" rpy="${pi} 0 ${pi}" />
   </joint>
-  <joint name="arm_1_base_link_z-joint_1" type="fixed">
-    <parent link="arm_1_base_link_z" />
-    <child link="arm_1_base_link" />
+  <joint name="right_base_link_z-joint_1" type="fixed">
+    <parent link="right_base_link_z" />
+    <child link="right_base_link" />
     <origin xyz="0 0 0" rpy="0 0 0" />
   </joint>
